File: KiCAD/3340VCO/3340VCO.kicad_pcb (KiCad board)
At the start: 2 copper layers, 81.9 x 99.1 mm, 74 parts, among them J1 ERK_PWR, J2 IN1, J3 IN2, J4 W_FORM, J5 TP_GND, J6 TP_GND, J7 OUT, SW1 SW_Rotary5, U1 NJM072D, U2 NJM072D, U3 NJM072D, U4 NJM072D, U5 AS3340

Commit message: 部品配置
Parts:
- added J8: OUT, Connector_JST:JST_XH_B2B-XH-A_1x02_P2.50mm_Vertical, F.Cu at (127.0, 139.7)
- J1: value ERK_PWR -> CV_IN; footprint Connector_IDC:IDC-Header_2x05_P2.54mm_Vertical -> Connector_JST:JST_XH_B2B-XH-A_1x02_P2.50mm_Vertical
- J2: value IN1 -> ERK_PWR; footprint Connector_JST:JST_XH_B6B-XH-A_1x06_P2.50mm_Vertical -> Connector_IDC:IDC-Header_2x05_P2.54mm_Vertical
- J3: value IN2 -> MOD_IN; footprint Connector_JST:JST_XH_B6B-XH-A_1x06_P2.50mm_Vertical -> Connector_JST:JST_XH_B4B-XH-A_1x04_P2.50mm_Vertical
- J4: value W_FORM -> IN2; footprint Connector_JST:JST_XH_B4B-XH-A_1x04_P2.50mm_Vertical -> Connector_JST:JST_XH_B6B-XH-A_1x06_P2.50mm_Vertical
- J5: value TP_GND -> W_FORM; footprint Connector_PinHeader_2.54mm:PinHeader_1x02_P2.54mm_Vertical -> Connector_JST:JST_XH_B4B-XH-A_1x04_P2.50mm_Vertical
- J7: value OUT -> TP_GND; footprint Connector_JST:JST_XH_B2B-XH-A_1x02_P2.50mm_Vertical -> Connector_PinHeader_2.54mm:PinHeader_1x02_P2.54mm_Vertical
- moved J7 82.0 mm to (130.8, 58.4)
- moved J5 77.7 mm to (116.2, 139.7), turned to 180 degrees
- moved J3 66.8 mm to (166.4, 102.9), turned to 90 degrees
- moved J1 55.8 mm to (141.6, 57.3), turned to 0 degrees
- moved J6 55.0 mm to (163.2, 144.8), turned to 180 degrees
- moved J4 41.5 mm to (155.0, 113.8), turned to 0 degrees
- moved C2 39.6 mm to (120.0, 76.8), turned to 180 degrees
- moved R7 33.4 mm to (114.9, 84.5)
- moved J2 31.2 mm to (110.6, 76.8), turned to 180 degrees
- moved D2 29.0 mm to (120.0, 84.5)
- moved D1 20.7 mm to (117.5, 59.1)
- moved C1 17.2 mm to (117.5, 66.7), turned to 0 degrees
- moved RV6 15.3 mm to (106.7, 99.7), turned to -90 degrees
- moved R6 13.3 mm to (104.8, 59.1)
- moved R30 12.1 mm to (146.1, 143.5)
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Connections:
- J1 pad 1: -12V -> CV
- J1 pad 2: -12V -> GND
- J2 pad 1: CV -> -12V
- J2 pad 2: GND -> -12V
- J2 pad 3: PWM -> GND
- J2 pad 5: MOD -> GND
- J3 pad 1: HARD_SYNC -> PWM
- J3 pad 3: SOFT_SYNC -> MOD
- J4 pad 1: SAW -> HARD_SYNC
- J4 pad 2: TRIANGLE -> GND
- J4 pad 3: PULSE -> SOFT_SYNC
- J4 pad 4: Net-(J4-Pad4) -> GND
- J5 pad 1: GND -> TRIANGLE
- J5 pad 2: GND -> SAW
- J7 pad 1: Net-(J7-Pad1) -> GND
- R28 pad 1: Net-(J4-Pad4) -> Net-(J5-Pad4)
- R29 pad 2: Net-(J7-Pad1) -> Net-(J8-Pad1)
- U2 pad 3: Net-(J4-Pad4) -> Net-(J5-Pad4)
Other:
- board size 81.9 x 99.1 mm -> 78.1 x 99.1 mm

Commit message: 基板製造
Parts:
- added G***: LOGO, myfootprint:Silk_PNPN_Manufactory_600dpi, F.Cu at (110.5, 115.6)
- added G***: LOGO, myfootprint:Silk_PNPN_Thyristor_1200dpi, F.Cu at (112.4, 121.3)
- added J9: TP_GND, Connector_PinHeader_2.54mm:PinHeader_1x02_P2.54mm_Vertical, F.Cu at (163.2, 141.6)
- added TP1: +5V, TestPoint:TestPoint_Pad_D1.0mm, F.Cu at (157.5, 121.3)
- moved J6 67.5 mm to (105.4, 109.9), turned to 90 degrees
- moved D1 2.55 mm to (120.0, 59.1), turned to 180 degrees
- moved D2 2.54 mm to (117.5, 84.5), turned to 0 degrees
- renumbered R11 to R10, R12 to R11, R14 to R12, R10 to R14, R18 to R15, R15 to R16, R20 to R17, R17 to R18, R23 to R19, R24 to R20, R25 to R21, R26 to R22, R19 to R23, R16 to R24, R21 to R25, R22 to R26
Routing:
- net -12V: track 0.00 -> 233.1 mm
- net +12V: track 0.00 -> 224.1 mm
- net +5V: track 0.00 -> 79.4 mm, vias 0 -> 1
- net Net-(RV4-Pad2): track 0.00 -> 56.8 mm
- net FINE: track 0.00 -> 53.7 mm
- net Net-(J5-Pad4): track 0.00 -> 44.6 mm
- net Net-(R16-Pad1): track 0.00 -> 41.8 mm
- net Net-(R4-Pad2): track 0.00 -> 39.9 mm
- net Net-(R10-Pad2): track 0.00 -> 37.7 mm
- net SAW: track 0.00 -> 36.0 mm
- net OCTAVE: track 0.00 -> 33.6 mm
- net Net-(R22-Pad2): track 0.00 -> 32.4 mm
- net Net-(U4-Pad5): track 0.00 -> 29.1 mm
- net Net-(C17-Pad1): track 0.00 -> 28.4 mm
- net PULSE: track 0.00 -> 27.0 mm
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- added copper zone on B.Cu, net GND
Other:
- board text added: "+5V"
- board text added: "+5V_ADJ"
- board text added: "-12V G G G +12V"
- board text added: "2023.07"
- board text added: "3340VCO"
- board text added: "COM PLS SAW TRI"
- board text added: "CV G"
- board text added: "CV_ADJ"
- board text added: "FINE"
- board text added: "G OUT"
- board text added: "GND"
- board text added: "HFREQ"
- board text added: "HSY G SSY G LFM G"
- board text added: "MOD"
- board text added: "OCTAVE"
- board text added: "OUT"
- board text added: "PULSE WIDTH"
- board text added: "PWM"
- board text added: "PWM G MOD G"
- board text added: "SCALE"
- board text added: "Ver.1.0"
- board text added: "WAV_FORM"
- board text added: "https://dad8893.blogspot.com/"

Commit message: '23夏コミケ
Parts:
- added TP2: +1V, TestPoint:TestPoint_Pad_D1.0mm, F.Cu at (169.5, 62.2)
- added TP3: OCT, TestPoint:TestPoint_Pad_D1.0mm, F.Cu at (151.8, 62.9)
- C12: value 1000pF -> 1000pF/PP
- C16: footprint Capacitor_THT:C_Rect_L7.0mm_W2.5mm_P5.00mm -> Capacitor_THT:C_Rect_L7.0mm_W3.5mm_P5.00mm
- J4: value IN2 -> EXT
- R15: value 220k -> 270k
- RV3: value 100k -> 50k
- RV7: value 50k -> 100k
- moved R1 12.7 mm to (154.3, 85.1)
- moved R5 12.7 mm to (154.3, 72.4)
- moved R2 6.35 mm to (154.3, 81.9)
- moved R4 6.35 mm to (154.3, 75.6)
- moved RV6 5.08 mm to (106.7, 94.6), turned to 90 degrees
- moved C16 0.26 mm to (153.7, 105.0)
Connections:
- R13 pad 1: Net-(R14-Pad2) -> Net-(R13-Pad1)
- R14 pad 2: Net-(R14-Pad2) -> Net-(R13-Pad1)
- RV4 pad 1: PWM -> Net-(RV4-Pad1)
- RV4 pad 3: Net-(RV4-Pad3) -> PWM
- RV6 pad 1: Net-(R14-Pad2) -> Net-(R12-Pad1)
- RV6 pad 2: Net-(R14-Pad2) -> Net-(R13-Pad1)
- RV6 pad 3: Net-(R12-Pad1) -> Net-(R13-Pad1)
- RV8 pad 1: MOD -> GND
- RV8 pad 3: GND -> MOD
- SW1 pad 10: (no net) -> GND
- SW1 pad 2: Net-(R1-Pad2) -> Net-(R4-Pad2)
- SW1 pad 3: Net-(R2-Pad2) -> Net-(R3-Pad2)
- SW1 pad 4: Net-(R3-Pad2) -> Net-(R2-Pad2)
- SW1 pad 5: Net-(R4-Pad2) -> Net-(R1-Pad2)
- SW1 pad 7: GND -> (no net)
- U3 pad 6: Net-(RV4-Pad3) -> Net-(RV4-Pad1)
- U3 pad 7: Net-(RV4-Pad3) -> Net-(RV4-Pad1)
- U5 pad 3: Net-(R14-Pad2) -> Net-(R13-Pad1)
Routing:
- net Net-(R14-Pad2): track 26.4 -> 0.00 mm
- net Net-(R13-Pad1): track 0.00 -> 26.4 mm
- net Net-(RV4-Pad3): track 18.3 -> 0.00 mm
- net +5V: track 79.4 -> 66.7 mm
- net Net-(RV4-Pad1): track 0.00 -> 12.3 mm
- net MOD: track 11.0 -> 19.9 mm
- net Net-(RV1-Pad3): track 20.9 -> 27.6 mm
- net OCTAVE: track 33.6 -> 39.4 mm
- net Net-(R4-Pad2): track 39.9 -> 34.2 mm
- net PWM: track 22.4 -> 17.4 mm
Other:
- board text added: "+1V"
- board text added: "OCT"
- board text added: "Ver.1.1"
- board text removed: "Ver.1.0"
