File: KiCAD/3340VCO/3340VCO.kicad_sch (KiCad schematic)
At the start: 74 parts, among them J1 ERK_PWR, J2 IN1, J3 IN2, J4 W_FORM, J5 TP_GND, J6 TP_GND, J7 OUT, SW1 SW_Rotary5, U1 NJM072D, U2 NJM072D, U3 NJM072D, U4 NJM072D, U5 AS3340

Commit message: 部品配置
Parts:
- removed J2: IN1, Connector_JST:JST_XH_B6B-XH-A_1x06_P2.50mm_Vertical, symbol Connector_Generic:Conn_01x06
- added J1: CV_IN, Connector_JST:JST_XH_B2B-XH-A_1x02_P2.50mm_Vertical, symbol Connector_Generic:Conn_01x02
- added J3: MOD_IN, Connector_JST:JST_XH_B4B-XH-A_1x04_P2.50mm_Vertical, symbol Connector_Generic:Conn_01x04
- renumbered J1 to J2, J3 to J4, J4 to J5, J5 to J6, J6 to J7, J7 to J8
Connections:
- net CV: now also J1.1 (Pin_1)
- net GND: now also J1.2 (Pin_2), J3.2 (Pin_2), J3.4 (Pin_4)
- net MOD: now also J3.3 (Pin_3)
- net PWM: now also J3.1 (Pin_1)
- net SAW: now also J5.2 (Pin_2); no longer J5.1 (Pin_1)
- net TRIANGLE: now also J5.1 (Pin_1); no longer J5.2 (Pin_2)

Commit message: 基板製造
Parts:
- added J9: TP_GND, Connector_PinHeader_2.54mm:PinHeader_1x02_P2.54mm_Vertical, symbol Connector_Generic:Conn_01x02
- added TP1: +5V, TestPoint:TestPoint_Pad_D1.0mm, symbol Connector:TestPoint
- renumbered R11 to R10, R12 to R11, R14 to R12, R10 to R14, R18 to R15, R15 to R16, R20 to R17, R17 to R18, R23 to R19, R24 to R20, R25 to R21, R26 to R22, R19 to R23, R16 to R24, R21 to R25, R22 to R26
Connections:
- net +5V: now also TP1.1
- net GND: now also J9.1 (Pin_1), J9.2 (Pin_2)

Commit message: '23夏コミケ
Parts:
- added TP2: +1V, TestPoint:TestPoint_Pad_D1.0mm, symbol Connector:TestPoint
- added TP3: OCT, TestPoint:TestPoint_Pad_D1.0mm, symbol Connector:TestPoint
- C12: value 1000pF -> 1000pF/PP
- C16: footprint Capacitor_THT:C_Rect_L7.0mm_W2.5mm_P5.00mm -> Capacitor_THT:C_Rect_L7.0mm_W3.5mm_P5.00mm
- J4: value IN2 -> EXT
- RV1: value 1k -> 10k/B
- RV3: value 100k -> 50k/B
- RV4, RV8: value 50k -> 50k/B
- RV7: value 50k -> 100k
Connections:
- net GND: now also RV8.1, SW1.10; no longer RV8.3, SW1.7
- net MOD: now also RV8.3; no longer RV8.1
- net OCTAVE: now also TP3.1
- net PWM: now also RV4.3; no longer RV4.1
- net at R13.1, R14.2, RV6.2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: now also RV6.3; no longer RV6.1
- net at R12.1: now also RV6.1; no longer RV6.3
- net at U3.6 (-), U3.7: now also RV4.1; no longer RV4.3
- net at R4.2, R5.1, U1.5 (+): now also SW1.2; no longer SW1.5
- net at R3.2, R4.1: now also SW1.3; no longer SW1.4
- net at R2.2, R3.1: now also SW1.4; no longer SW1.3
- net at RV1.3, U1.6 (-), U1.7: now also TP2.1
- net at R1.2, R2.1: now also SW1.5; no longer SW1.2
Other:
- moved on the sheet: RV3, RV6, RV8, U3B
